File: ic2RJ45.sch (KiCad schematic (older format))
At the start: 7 parts, among them J1 RJ45, P1 POT, P2 TERM, P3 .

Commit message: further design modifications
Parts:
- CONN1: footprint (none) -> IC_CONN_02x09:IC_CONN_02x09
- CONN2: footprint (none) -> IC_CONN_02x09_axial:IC_CONN_02x09_axial
- J1: footprint (none) -> RJ45_Pollin:RJ45_Pollin
- P1: footprint (none) -> Pin_Headers:Pin_Header_Straight_1x03
- P2: footprint (none) -> Pin_Headers:Pin_Header_Straight_2x01
- P3: footprint (none) -> Pin_Headers:Pin_Header_Straight_1x08
- R1: footprint (none) -> Resistors_Universal:Resistor_SMDuniversal_0805to1206_HandSoldering
Connections:
- net GND: now also J1.9 (SHIELD), P1.1 (P1); no longer P1.2 (P2)
- net at CONN1.12 (Tankgeber_2_?), CONN2.12 (Tankgeber_2_?): now also P1.2 (P2); no longer P1.1 (P1)
- net at CONN2.7 (Feststellbremse_?): now also CONN1.7 (Feststellbremse_?)
- no-connect marks 9 -> 6
Changed lines of the file:
@@
 F 0 "CONN2" H 5200 2850 60  0000 C CNN
 F 1 "IC_Golf7" H 5200 3850 60  0000 C CNN
-F 2 "" H 5200 2750 60  0000 C CNN
+F 2 "IC_CONN_02x09_axial:IC_CONN_02x09_axial" H 5200 2750 60  0001 C CNN
 F 3 "" H 5200 2750 60  0000 C CNN
 	1    5250 3350
@@
 F 0 "J1" H 5400 2100 60  0000 C CNN
 F 1 "RJ45" H 5050 2100 60  0000 C CNN
-F 2 "" H 5200 1600 60  0000 C CNN
+F 2 "RJ45_Pollin:RJ45_Pollin" H 5200 1600 60  0001 C CNN
 F 3 "" H 5200 1600 60  0000 C CNN
 	1    5200 1600
@@
 F 0 "P2" H 4350 2900 50  0000 C CNN
 F 1 "TERM" V 4450 2750 50  0000 C CNN
-F 2 "" H 4350 2750 60  0000 C CNN
+F 2 "Pin_Headers:Pin_Header_Straight_2x01" H 4350 2750 60  0001 C CNN
 F 3 "" H 4350 2750 60  0000 C CNN
 	1    4350 2750
@@
 F 0 "R1" V 4230 2950 50  0000 C CNN
 F 1 "120" V 4150 2950 50  0000 C CNN
-F 2 "" V 4080 2950 30  0000 C CNN
+F 2 "Resistors_Universal:Resistor_SMDuniversal_0805to1206_HandSoldering" V 4080 2950 30  0001 C CNN
 F 3 "" H 4150 2950 30  0000 C CNN
 	1    4150 2950
@@
 Wire Wire Line
 	4400 2950 4550 2950
-$Comp
-L CONN_01X03 P1
-U 1 1 5891FC6C
-P 4100 3550
-F 0 "P1" H 4100 3750 50  0000 C CNN
-F 1 "POT" V 4200 3550 50  0000 C CNN
-F 2 "" H 4100 3550 60  0000 C CNN
-F 3 "" H 4100 3550 60  0000 C CNN
-	1    4100 3550
-	-1   0    0    1
-$EndComp
-Wire Wire Line
-	3950 3550 4400 3550
-Wire Wire Line
-	4400 3550 4400 3650
-Wire Wire Line
-	4400 3650 4550 3650
-Wire Wire Line
-	4000 3650 4350 3650
-Wire Wire Line
-	4350 3650 4350 3600
-Wire Wire Line
-	4350 3600 4450 3600
-Wire Wire Line
-	4450 3600 4450 3550
-Wire Wire Line
-	4450 3550 4550 3550
 Wire Wire Line
 	3650 3450 4550 3450
@@
 Connection ~ 4550 2950
 $Comp
-L GND #PWR1
+L GND #PWR01
 U 1 1 5891FDC6
 P 4550 3750
-F 0 "#PWR1" H 4550 3500 50  0001 C CNN
+F 0 "#PWR01" H 4550 3500 50  0001 C CNN
 F 1 "GND" H 4550 3600 50  0000 C CNN
 F 2 "" H 4550 3750 60  0000 C CNN
@@
 $EndComp
 $Comp
-L GND #PWR2
+L GND #PWR02
 U 1 1 5891FDE7
 P 5050 2450
-F 0 "#PWR2" H 5050 2200 50  0001 C CNN
+F 0 "#PWR02" H 5050 2200 50  0001 C CNN
 F 1 "GND" H 5050 2300 50  0000 C CNN
 F 2 "" H 5050 2450 60  0000 C CNN
@@
 $EndComp
 $Comp
-L GND #PWR3
+L GND #PWR03
 U 1 1 5891FE01
 P 5350 2450
-F 0 "#PWR3" H 5350 2200 50  0001 C CNN
+F 0 "#PWR03" H 5350 2200 50  0001 C CNN
 F 1 "GND" H 5350 2300 50  0000 C CNN
 F 2 "" H 5350 2450 60  0000 C CNN
@@
 $EndComp
 $Comp
-L VCC #PWR4
+L VCC #PWR04
 U 1 1 5891FE64
 P 5550 2450
-F 0 "#PWR4" H 5550 2300 50  0001 C CNN
+F 0 "#PWR04" H 5550 2300 50  0001 C CNN
 F 1 "VCC" H 5550 2600 50  0000 C CNN
 F 2 "" H 5550 2450 60  0000 C CNN
@@
 $EndComp
 $Comp
-L VCC #PWR5
+L VCC #PWR05
 U 1 1 5891FE85
 P 5900 3750
-F 0 "#PWR5" H 5900 3600 50  0001 C CNN
+F 0 "#PWR05" H 5900 3600 50  0001 C CNN
 F 1 "VCC" H 5900 3900 50  0000 C CNN
 F 2 "" H 5900 3750 60  0000 C CNN
@@
 F 0 "P3" H 5200 2700 50  0000 C CNN
 F 1 "." V 5300 2250 50  0000 C CNN
-F 2 "" H 5200 2250 60  0000 C CNN
+F 2 "Pin_Headers:Pin_Header_Straight_1x08" H 5200 2250 60  0001 C CNN
 F 3 "" H 5200 2250 60  0000 C CNN
 	1    5200 2250
@@
 Connection ~ 5150 2450
 Connection ~ 5050 2450
-NoConn ~ 5750 1250
 $Comp
 L IC_Golf7 CONN1
@@
 F 0 "CONN1" H 2900 2850 60  0000 C CNN
 F 1 "IC_Golf7" H 2900 3850 60  0000 C CNN
-F 2 "" H 2900 2750 60  0000 C CNN
+F 2 "IC_CONN_02x09:IC_CONN_02x09" H 2900 2750 60  0001 C CNN
 F 3 "" H 2900 2750 60  0000 C CNN
 	1    2950 3350
@@
 Wire Wire Line
 	3650 3350 4550 3350
-Connection ~ 4300 3450
-Wire Wire Line
-	3950 3550 3950 3650
-Wire Wire Line
-	3950 3650 3650 3650
-Connection ~ 4300 3550
-Wire Wire Line
-	3650 3550 3900 3550
-Wire Wire Line
-	3900 3550 3900 3600
-Wire Wire Line
-	3900 3600 4000 3600
-Wire Wire Line
-	4000 3600 4000 3650
-Connection ~ 4300 3650
+Wire Wire Line
+	3650 3550 4550 3550
 Wire Wire Line
 	4550 3750 3650 3750
@@
 Wire Wire Line
 	2100 2950 2300 2950
-NoConn ~ 5900 3150
 NoConn ~ 5900 3250
 NoConn ~ 5900 3550
 NoConn ~ 5900 3650
-NoConn ~ 2300 3150
 NoConn ~ 2300 3250
 NoConn ~ 2300 3550
 NoConn ~ 2300 3650
+Wire Wire Line
+	5900 3150 6200 3150
+Wire Wire Line
+	6200 3150 6200 4200
+Wire Wire Line
+	6200 4200 2050 4200
+Wire Wire Line
+	2050 4200 2050 3150
+Wire Wire Line
+	2050 3150 2300 3150
+$Comp
+L CONN_01X03 P1
+U 1 1 5891FC6C
+P 4100 3550
+F 0 "P1" H 4100 3750 50  0000 C CNN
+F 1 "POT" V 4200 3550 50  0000 C CNN
+F 2 "Pin_Headers:Pin_Header_Straight_1x03" H 4100 3550 60  0001 C CNN
+F 3 "" H 4100 3550 60  0000 C CNN
+	1    4100 3550
+	-1   0    0    1
+$EndComp
+Connection ~ 4300 3550
+Wire Wire Line
+	3650 3650 4550 3650
+Connection ~ 4300 3650
+Connection ~ 4300 3450
+$Comp
+L GND #PWR?
+U 1 1 58923DD3
+P 5750 1250
+F 0 "#PWR?" H 5750 1000 50  0001 C CNN
+F 1 "GND" H 5750 1100 50  0000 C CNN
+F 2 "" H 5750 1250 60  0000 C CNN
+F 3 "" H 5750 1250 60  0000 C CNN
+	1    5750 1250
+	1    0    0    -1
+$EndComp
 $EndSCHEMATC
