File: ic2RJ45.kicad_pcb (KiCad board)
At the start: 2 copper layers, 47.5 x 27.9 mm, 7 parts, among them J1 RJ45, P1 ., P3 .

Commit message: finalized v1.1
Other:
- board text added: "github.com /mediadon/kicad_ic2RJ45"
- board text added: "v1.1"
- board text added: "© Daniel Laffling 2017"
Changed lines of the file:
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@@
     (area 23.800999 23.546999 71.449001 51.637001)
     (thickness 1.6)
-    (drawings 14)
+    (drawings 17)
     (tracks 78)
     (zones 0)
@@
   )
   (setup
-    (last_trace_width 0.43)
+    (last_trace_width 0.25)
     (user_trace_width 0.3)
     (user_trace_width 0.4)
@@
       (net 16 "Net-(CONN1-Pad17)"))
   )
+  (gr_text "© Daniel Laffling 2017" (at 36.322 37.592 90) (layer B.SilkS)
+    (effects (font (size 1 1) (thickness 0.2)) (justify mirror))
+  )
+  (gr_text "github.com\n/mediadon/kicad_ic2RJ45" (at 31.496 37.592 90) (layer B.SilkS)
+    (effects (font (size 1 1) (thickness 0.2)) (justify mirror))
+  )
+  (gr_text v1.1 (at 34.036 37.592 90) (layer B.SilkS)
+    (effects (font (size 1 1) (thickness 0.2)) (justify mirror))
+  )
   (dimension 27.94 (width 0.3) (layer Eco1.User)
